File: cdu-hat.kicad_pcb (KiCad board)
At the start: 6 copper layers, 65 x 44.7 mm, 5 parts, among them J3 Conn_02x20_Odd_Even

Commit message: Migrated to new kicad version
Other:
- net class Default removed
